File: schematics/Sketching2025badge/Sketching2025badge.kicad_pcb (KiCad board)
At the start: 2 copper layers, 100 x 100 mm, 47 parts, among them CN1 X6511FRS-04-C85D30, J1 Conn_02x03, SW1 Capacitive_Button, SW10 SSSS811101, SW2 Capacitive_Button, SW3 Capacitive_Button, U1 ATtiny816-M

Commit message: update with prelim version sent to PCBWay
Parts:
- moved D1 13.5 mm to (108.8, 56.2)
- moved R8 8.94 mm to (108.8, 72.2)
- moved R1 2.79 mm to (137.2, 110.6)
- moved R2 2.79 mm to (137.2, 113.8)
Routing:
- net Net-(D1-A): track 4.01 -> 16.0 mm
- net /LED: track 108.3 -> 115.9 mm
- net GND: track 412.4 -> 417.8 mm
- net /SCL: track 64.1 -> 68.5 mm
- net /SDA: track 63.3 -> 66.1 mm
- net Net-(LED6-DOUT): track 53.8 -> 52.5 mm
- net /RXD: track 64.9 -> 63.8 mm
Other:
- board text added: "31 Aug 2025 - @todbot & @leeborg github.com/todbot/Sketching2025badge"
- board text added: "SAO"
- board text added: "leddat"
- board text added: "pa1"
- board text added: "pa2"
- board text added: "pb2"
- board text added: "pb3"
- board text removed: "29 Aug 2025 - @todbot & @leeborg github.com/todbot/Sketching2025badge"
